Commit message: Update rsc folder

File: rsc/huskyDemo/urdf/husky.urdf (robot description, URDF)
Before this commit: robot husky_robot, 11 links, 10 joints
Links:
- removed link imu_link
- added link depth_camera_front_camera, mass 0.16043; visual mesh filename=package://anymal_c_simple_description/meshes/depth_camera.d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 scale=1.0 1.0 1.0
- added link depth_camera_front_camera_parent
- added link depth_camera_front_color_frame
- added link depth_camera_front_color_optical_frame
- added link depth_camera_front_depth_optical_frame
- added link depth_camera_rear_camera, mass 0.16043; visual mesh filename=package://anymal_c_simple_description/meshes/depth_camera.d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 scale=1.0 1.0 1.0
- added link depth_camera_rear_camera_parent
- added link depth_camera_rear_color_frame
- added link depth_camera_rear_color_optical_frame
- added link depth_camera_rear_depth_optical_frame
Joints:
- removed joint imu_joint
- added joint depth_camera_front_camera_joint: type fixed, parent base_link, child depth_camera_front_camera, origin xyz=-0.2 0 0.309 rpy=0 0.31415926535 3.14159
- added joint depth_camera_front_camera_parent_to_color_frame: type fixed, parent depth_camera_front_camera_parent, child depth_camera_front_color_frame, origin xyz=0 0.015 0 rpy=0 0 0
- added joint depth_camera_front_camera_parent_to_depth_optical_frame: type fixed, parent depth_camera_front_camera_parent, child depth_camera_front_depth_optical_frame, origin xyz=0.0 0.0 0.0 rpy=-1.57079632679 0.0 -1.57079632679
- added joint depth_camera_front_camera_to_camera_parent: type fixed, parent depth_camera_front_camera, child depth_camera_front_camera_parent, origin xyz=0.0255 0.0175 0.0 rpy=0.0 0.0 0.0
- added joint depth_camera_front_color_frame_to_color_optical_frame: type fixed, parent depth_camera_front_color_frame, child depth_camera_front_color_optical_frame, origin xyz=0.0 0.0 0.0 rpy=-1.57079632679 0.0 -1.57079632679
- added joint depth_camera_rear_camera_joint: type fixed, parent base_link, child depth_camera_rear_camera, origin xyz=0.2 0 0.309 rpy=0 0.31415926535 0
- added joint depth_camera_rear_camera_parent_to_color_frame: type fixed, parent depth_camera_rear_camera_parent, child depth_camera_rear_color_frame, origin xyz=0 0.015 0 rpy=0 0 0
- added joint depth_camera_rear_camera_parent_to_depth_optical_frame: type fixed, parent depth_camera_rear_camera_parent, child depth_camera_rear_depth_optical_frame, origin xyz=0.0 0.0 0.0 rpy=-1.57079632679 0.0 -1.57079632679
- added joint depth_camera_rear_camera_to_camera_parent: type fixed, parent depth_camera_rear_camera, child depth_camera_rear_camera_parent, origin xyz=0.0255 0.0175 0.0 rpy=0.0 0.0 0.0
- added joint depth_camera_rear_color_frame_to_color_optical_frame: type fixed, parent depth_camera_rear_color_frame, child depth_camera_rear_color_optical_frame, origin xyz=0.0 0.0 0.0 rpy=-1.57079632679 0.0 -1.57079632679
