Commit message: Upgrade rsc folder

File: rsc/kanga/urdf/kangaSensors.urdf (robot description, URDF)
Before this commit: robot onshape, 11 links, 10 joints
Links:
- added link antenna, mass 0.2000000000000000111; visual mesh filename=meshes/antenna.obj
- added link camera_above_camera, mass 0.16043; visual mesh filename=package://anymal_c_simple_description/meshes/depth_camera.d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 scale=1.0 1.0 1.0
- added link camera_above_camera_parent
- added link camera_above_color_frame
- added link camera_above_color_optical_frame
- added link camera_above_optical_frame
- added link camera_below_camera, mass 0.16043; visual mesh filename=package://anymal_c_simple_description/meshes/depth_camera.d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 scale=1.0 1.0 1.0
- added link camera_below_camera_parent
- added link camera_below_color_frame
- added link camera_below_color_optical_frame
- added link camera_below_optical_frame
- added link camera_front_camera, mass 0.16043; visual mesh filename=package://anymal_c_simple_description/meshes/depth_camera.d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 scale=1.0 1.0 1.0
- added link camera_front_camera_parent
- added link camera_front_color_frame
- added link camera_front_color_optical_frame
- added link camera_front_optical_frame
- added link camera_rear_camera, mass 0.16043; visual mesh filename=package://anymal_c_simple_description/meshes/depth_camera.d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 scale=1.0 1.0 1.0
- added link camera_rear_camera_parent
- added link camera_rear_color_frame
- added link camera_rear_color_optical_frame
- added link camera_rear_optical_frame
- added link composite_part_1, mass 5; visual mesh filename=meshes/composite_part_1.obj
- added link imu_camera, mass 0.16043; visual mesh filename=package://anymal_c_simple_description/meshes/depth_camera.d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 scale=1.0 1.0 1.0
- added link imu_camera_parent
- added link imu_color_frame
- added link imu_color_optical_frame
- added link imu_optical_frame
- added link radio, mass 0.2000000000000000111; visual mesh filename=meshes/radio.obj
Joints:
- added joint antennaMount: type fixed, parent radio, child antenna, origin xyz=0 0 -0.095 rpy=1.6028614105982569444e-17 -2.7755575615628923371e-16 1.570796326794896558, axis 0 0 1, limit effort=1 velocity=20
- added joint batteryBox: type fixed, parent body, child composite_part_1, origin xyz=-0.1426882932794905634 0.23373218016369090577 -0.14420437190083026935 rpy=1.57079632679489678 -0 -1.570796326794896558, axis 0 0 1, limit effort=1 velocity=20
- added joint camera_above_camera_joint: type fixed, parent body, child camera_above_camera, origin xyz=-0.135 0.52 0.81 rpy=0.0 0.75 -1.45
- added joint camera_above_camera_parent_to_color_frame: type fixed, parent camera_above_camera_parent, child camera_above_color_frame, origin xyz=0 0.015 0 rpy=0 0 0
- added joint camera_above_camera_parent_to_optical_frame: type fixed, parent camera_above_camera_parent, child camera_above_optical_frame, origin xyz=0.0 0.0 0.0 rpy=-1.57079632679 0.0 -1.57079632679
- added joint camera_above_camera_to_camera_parent: type fixed, parent camera_above_camera, child camera_above_camera_parent, origin xyz=0.0255 0.0175 0.0 rpy=0.0 0.0 0.0
- added joint camera_above_color_frame_to_color_optical_frame: type fixed, parent camera_above_color_frame, child camera_above_color_optical_frame, origin xyz=0.0 0.0 0.0 rpy=-1.57079632679 0.0 -1.57079632679
- added joint camera_below_camera_joint: type fixed, parent body, child camera_below_camera, origin xyz=-0.01371171  0.18 -0.24 rpy=1.57079632679 1.57079632679 1.57079632679
- added joint camera_below_camera_parent_to_color_frame: type fixed, parent camera_below_camera_parent, child camera_below_color_frame, origin xyz=0 0.015 0 rpy=0 0 0
- added joint camera_below_camera_parent_to_optical_frame: type fixed, parent camera_below_camera_parent, child camera_below_optical_frame, origin xyz=0.0 0.0 0.0 rpy=-1.57079632679 0.0 -1.57079632679
- added joint camera_below_camera_to_camera_parent: type fixed, parent camera_below_camera, child camera_below_camera_parent, origin xyz=0.0255 0.0175 0.0 rpy=0.0 0.0 0.0
- added joint camera_below_color_frame_to_color_optical_frame: type fixed, parent camera_below_color_frame, child camera_below_color_optical_frame, origin xyz=0.0 0.0 0.0 rpy=-1.57079632679 0.0 -1.57079632679
- added joint camera_front_camera_joint: type fixed, parent body, child camera_front_camera, origin xyz=-0.01371171  -0.06 -0.19 rpy=0 0.31415926535 -1.57079632679
- added joint camera_front_camera_parent_to_color_frame: type fixed, parent camera_front_camera_parent, child camera_front_color_frame, origin xyz=0 0.015 0 rpy=0 0 0
- added joint camera_front_camera_parent_to_optical_frame: type fixed, parent camera_front_camera_parent, child camera_front_optical_frame, origin xyz=0.0 0.0 0.0 rpy=-1.57079632679 0.0 -1.57079632679
- added joint camera_front_camera_to_camera_parent: type fixed, parent camera_front_camera, child camera_front_camera_parent, origin xyz=0.0255 0.0175 0.0 rpy=0.0 0.0 0.0
- added joint camera_front_color_frame_to_color_optical_frame: type fixed, parent camera_front_color_frame, child camera_front_color_optical_frame, origin xyz=0.0 0.0 0.0 rpy=-1.57079632679 0.0 -1.57079632679
- added joint camera_rear_camera_joint: type fixed, parent body, child camera_rear_camera, origin xyz=-0.01371171  0.5 -0.19 rpy=0 0.31415926535 1.57079632679
- added joint camera_rear_camera_parent_to_color_frame: type fixed, parent camera_rear_camera_parent, child camera_rear_color_frame, origin xyz=0 0.015 0 rpy=0 0 0
- added joint camera_rear_camera_parent_to_optical_frame: type fixed, parent camera_rear_camera_parent, child camera_rear_optical_frame, origin xyz=0.0 0.0 0.0 rpy=-1.57079632679 0.0 -1.57079632679
- added joint camera_rear_camera_to_camera_parent: type fixed, parent camera_rear_camera, child camera_rear_camera_parent, origin xyz=0.0255 0.0175 0.0 rpy=0.0 0.0 0.0
- added joint camera_rear_color_frame_to_color_optical_frame: type fixed, parent camera_rear_color_frame, child camera_rear_color_optical_frame, origin xyz=0.0 0.0 0.0 rpy=-1.57079632679 0.0 -1.57079632679
- added joint imu_camera_joint: type fixed, parent body, child imu_camera, origin xyz=-0.01371171  0.18 -0.18 rpy=0.0 0.0 1.57079632679
- added joint imu_camera_parent_to_color_frame: type fixed, parent imu_camera_parent, child imu_color_frame, origin xyz=0 0.015 0 rpy=0 0 0
- added joint imu_camera_parent_to_optical_frame: type fixed, parent imu_camera_parent, child imu_optical_frame, origin xyz=0.0 0.0 0.0 rpy=-1.57079632679 0.0 -1.57079632679
- added joint imu_camera_to_camera_parent: type fixed, parent imu_camera, child imu_camera_parent, origin xyz=0.0255 0.0175 0.0 rpy=0.0 0.0 0.0
- added joint imu_color_frame_to_color_optical_frame: type fixed, parent imu_color_frame, child imu_color_optical_frame, origin xyz=0.0 0.0 0.0 rpy=-1.57079632679 0.0 -1.57079632679
- added joint radioMount: type fixed, parent body, child radio, origin xyz=-0.14 0.51 -0.22 rpy=3.141592653589793116 -0 1.570796326794896558, axis 0 0 1, limit effort=1 velocity=20
- joint suspension_left: limit lower=-0.34906585039886589561 upper=0.34906585039886589561 effort=100 velocity=20 -> lower=-0.52359877559  upper=0.52359877559  effort=100 velocity=20; type fixed -> revolute
- joint suspension_right: limit lower=-0.34906585039886589561 upper=0.34906585039886589561 effort=100 velocity=20 -> lower=-0.52359877559  upper=0.52359877559  effort=100 velocity=20; type fixed -> revolute

Commit message: update intrinsic documentation

File: rsc/kanga/urdf/kangaSensors.urdf (robot description, URDF)
Before this commit: robot onshape, 39 links, 38 joints
Joints:
- joint camera_front_camera_joint: origin xyz=-0.01371171  -0.06 -0.19 rpy=0 0.31415926535 -1.57079632679 -> xyz=-0.01371171  -0.06 -0.19 rpy=0 0.26179938779  -1.57079632679
